File: 3ChannelCCdriver/3ChannelCCdriver.kicad_sch (KiCad schematic)
At the start: 8 parts, among them J2 Screw_Terminal_01x02, J3 Screw_Terminal_01x02, J4 Screw_Terminal_01x02, J5 Screw_Terminal_01x02

Commit message: Added documentation
Parts:
- J3, J4, J5: LCSC (none) -> C2922597
Changed lines of the file:
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@@
       (effects (font (size 1.27 1.27)) hide)
     )
-    (property "Datasheet" "~" (at 223.52 68.58 0)
+    (property "Datasheet" "https://datasheet.lcsc.com/lcsc/2112021230_JILN-JL308-25402G01_C2922597.pdf" (at 223.52 68.58 0)
+      (effects (font (size 1.27 1.27)) hide)
+    )
+    (property "LCSC" "C2922597" (at 223.52 68.58 0)
       (effects (font (size 1.27 1.27)) hide)
     )
@@
       (effects (font (size 1.27 1.27)) hide)
     )
-    (property "Datasheet" "~" (at 223.52 93.98 0)
+    (property "Datasheet" "https://datasheet.lcsc.com/lcsc/2112021230_JILN-JL308-25402G01_C2922597.pdf" (at 223.52 93.98 0)
+      (effects (font (size 1.27 1.27)) hide)
+    )
+    (property "LCSC" "C2922597" (at 223.52 93.98 0)
       (effects (font (size 1.27 1.27)) hide)
     )
@@
       (effects (font (size 1.27 1.27)) hide)
     )
-    (property "Datasheet" "~" (at 223.52 42.545 0)
+    (property "Datasheet" "https://datasheet.lcsc.com/lcsc/2112021230_JILN-JL308-25402G01_C2922597.pdf" (at 223.52 42.545 0)
       (effects (font (size 1.27 1.27)) hide)
     )
+    (property "LCSC" "C2922597" (at 223.52 42.545 0)
+      (effects (font (size 1.27 1.27)) hide)
+    )

Commit message: neat-ified schematics
Parts:
- J2: value Screw_Terminal_01x02 -> 1x02ScrewTerminal_P5.08mm
Other:
- note added: "CHANGELOG/NOTES REV A: Initial Design Rev B: Edited CC LED driver to edit the diode placement. Rev A had an incorrect diode schematic Also added R/C filter to DIM input to soft start the signal and prevent the pull-up from causing a flash on startup"
- note removed: "CHANGELOG/NOTES REV A:"
